File: vector_gen/vector_gen.sch (KiCad schematic (older format))
At the start: 59 parts, among them U1 LM2904, U10 MCP4922, U11 MCP4922, U12 4019, U13 LM336, U2 Y3014B, U3 Y3014B, U4 MCP6292, U5 4066, U6 LF412, U7 TL072IP, U8 TL072IP, U9 LM319

Commit message: More additions.
Parts:
- added C? (x3): .1u, symbol Device:C
- added C? (x4): 1u, symbol Device:C
- added J?: Conn_01x20_Female, symbol Connector:Conn_01x20_Female
- added R? (x3): 100k, symbol Device:R
- added R?: 15k, symbol Device:R
- added TP? (x16): TestPoint, TestPoint:TestPoint_THTPad_2.5x2.5mm_Drill1.2mm, symbol Connector:TestPoint
- added unit 2 of U1
- added unit 4 of U14
- added unit 3 of U14
- added unit 2 of U14
- added unit 5 of U14
- added U15, U16, U17: 74LS07, symbol 74xx:74LS07
- R?: value 22k -> 10k
- gave numbers to parts that had none: 1
Connections:
- net +5V: now also C?.1, C?.1, C?.1, C?.2, U14.14 (VCC), U15.14 (VCC), U16.14 (VCC), U17.14 (VCC)
- net -5V: now also R?.1
- net GND: now also C?.1, C?.1, C?.1, C?.1, C?.2, C?.2, C?.2, R?.1, R?.1, R?.1, U14.10, U14.12, U14.13, U14.4, U14.5, U14.7 (GND), U14.9, U15.7 (GND), U16.7 (GND), U17.7 (GND); no longer R?.2, RV?.3, U1.3 (+), U13.2 (+)
- net at R?.2, U4.1, U4.2 (-): now also TP?.1
- net at R?.2, R?.2, R?.2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: now also TP?.1; no longer U9.4 (+)
- net at R?.2, U4.6 (-), U4.7: now also TP?.1
- net at J?.5 (Pin_5), U5.5: now also U15.10
- net at J?.6 (Pin_6), U5.6: now also U15.12
- net at J?.4 (Pin_4), U2.3 (LOAD), U3.3 (LOAD): now also U15.8
- net at J?.1 (Pin_1), U2.4 (SD): now also U15.2
- net at U2.7 (Rb): now also C?.2
- net at J?.3 (Pin_3), U2.CLOCK (5), U3.CLOCK (5): now also U15.6
- net at J?.2 (Pin_2), U3.4 (SD): now also U15.4
- net at U3.7 (Rb): now also C?.2
- net at C?.1, R?.2, U5.2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: now also U9.4 (+), TP?.1
- net at J?.7 (Pin_7), U5.13: now also U16.2
- net at R?.2, U10.10 (VB): now also TP?.1
- net at R?.2, U10.14 (VA): now also TP?.1
- net at J?.11 (Pin_11), U10.3 (~CS): now also U16.10
- net at J?.9 (Pin_9), U10.4 (SCK), U11.4 (SCK): now also U16.6
- net at J?.10 (Pin_10), U10.5 (SDI), U11.5 (SDI): now also U16.8
- net at U11.10 (VB), U9.10 (-): now also TP?.1
- net at U11.14 (VA), U9.5 (-): now also TP?.1
- net at J?.12 (Pin_12), U11.3 (~CS): now also U16.12
- net at C?.1, R?.2, U5.10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: now also TP?.1
- net at J?.8 (Pin_8), U5.12: now also U16.4
- net at C?.1, R?.1, R?.2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: now also TP?.1 (x2)
- net at J?.13 (Pin_13), U12.9 (SA): now also U17.2
- net at J?.14 (Pin_14), U12.14 (SB): now also U17.4
- net at J?.15 (Pin_15), U14.1: now also U17.6
- net at J?.16 (Pin_16): now also U17.8
- net at J?.17 (Pin_17): now also U17.10
- net at J?.18 (Pin_18): now also U17.12
- net at J?.20 (Pin_20), U12.10 (Q0): now also J?.20 (Pin_20), TP?.1
- net at C?.1, R?.1, U8.1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: now also TP?.1
- net at C?.1, R?.1, U8.7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: now also TP?.1
- net at R?.2, RV?.1: now also Q?.2 (B), RV?.2
- net at R?.1, U14.3: now also TP?.1
- net at Q?.1 (E), R?.2, ZOUT.1 (In): now also TP?.1
- new net: C?.2, R?.2, U1.3 (+), U1.5 (+), U13.2 (+)
- new net: U1.6 (-), U1.7
- new net: R?.2, U14.11
- new net: R?.2, U14.8
- new net: R?.2, U14.6
- new net: R?.2, RV?.3
- new net: J?.1 (Pin_1), U15.1
- new net: J?.10 (Pin_10), U16.9
- new net: J?.11 (Pin_11), U16.11
- new net: J?.12 (Pin_12), U16.13
- new net: J?.13 (Pin_13), U17.1
- new net: J?.14 (Pin_14), U17.3
- new net: J?.15 (Pin_15), U17.5
- new net: J?.16 (Pin_16), U17.9
- new net: J?.17 (Pin_17), U17.11
- new net: J?.18 (Pin_18), U17.13
- new net: J?.2 (Pin_2), U15.3
- new net: J?.3 (Pin_3), U15.5
- new net: J?.4 (Pin_4), U15.9
- new net: J?.5 (Pin_5), U15.11
- new net: J?.6 (Pin_6), U15.13
- new net: J?.7 (Pin_7), U16.1
- new net: J?.8 (Pin_8), U16.3
- new net: J?.9 (Pin_9), U16.5
Other:
- note added: "3.3V DIGITAL INPUTS\n(PIN 20 IS 5V OUTPUT)"
- note added: "5V DIGITAL INPUTS (PIN 20 OUTPUT)"
- note added: "COEFFICIENT DAC BUFFERS"
- note added: "HOLD"
- note added: "PIN 20 MUST BE 5V \nTOLERANT INPUT"
- note added: "RESET"
- note added: "or 15k"
- moved on the sheet: U13

Commit message: Update with analog option connector, power connector, etc.
Parts:
- removed C? (x2): 1u, symbol Device:C
- removed R?: 15k, symbol Device:R
- added C10, C15, C16, C8, C9: 1u, symbol Device:C
- added J1: Conn_01x06_Female, symbol Connector:Conn_01x06_Female
- added J4: Conn_01x04_Male, symbol Connector:Conn_01x04_Male
- added RN1, RN2: R_Network09_US, Resistor_THT:R_Array_SIP10, symbol Device:R_Network09_US
- R21: renamed from R?; value 6.8k -> 22k
- U6: value LF412 -> LF412CP
- U6: value TL072IP -> LF412CP
- gave numbers to parts that had none: 66
- renumbered XOUT to XOUT1, YOUT to YOUT1, ZOUT to ZOUT1
Connections:
- net +5V: now also C15.2, J4.4 (Pin_4), RN1.1 (common), RN2.1 (common); no longer Q1.3 (C)
- net -5V: now also C16.1, J4.3 (Pin_3)
- net GND: now also J2.19 (Pin_19), J3.19 (Pin_19), RV1.3, C10.2, C15.1, C16.2, C8.2, C9.1, J1.6 (Pin_6), J4.1 (Pin_1); no longer U1.4 (V-), U4.4 (V-), U5.7 (VSS), U6.4 (V-)
- net at R2.2, TP2.1, U4.1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: now also J1.2 (Pin_2)
- net at R11.2, R4.2, R6.2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: now also J1.1 (Pin_1)
- net at R3.2, TP3.1, U4.6 (-)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: now also J1.3 (Pin_3)
- net at J2.5 (Pin_5), U15.10, U5.5: now also RN1.6 (R5)
- net at J2.6 (Pin_6), U15.12, U5.6: now also RN1.7 (R6)
- net at J2.4 (Pin_4), U15.8, U2.3 (LOAD)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: now also RN1.5 (R4)
- net at J2.1 (Pin_1), U15.2, U2.4 (SD): now also RN1.2 (R1)
- net at J2.3 (Pin_3), U15.6, U2.CLOCK (5)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: now also RN1.4 (R3)
- net at J2.2 (Pin_2), U15.4, U3.4 (SD): now also RN1.3 (R2)
- net at C11.1, R8.2, TP4.1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: now also J1.4 (Pin_4)
- net at J2.7 (Pin_7), U16.2, U5.13: now also RN1.8 (R7)
- net at J2.11 (Pin_11), U10.3 (~CS), U16.10: now also RN2.3 (R2)
- net at J2.9 (Pin_9), U10.4 (SCK), U11.4 (SCK)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: now also RN1.10 (R9)
- net at J2.10 (Pin_10), U10.5 (SDI), U11.5 (SDI)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: now also RN2.2 (R1)
- net at J2.12 (Pin_12), U11.3 (~CS), U16.12: now also RN2.4 (R3)
- net at C12.1, R10.2, TP5.1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: now also J1.5 (Pin_5)
- net at J2.8 (Pin_8), U16.4, U5.12: now also RN1.9 (R8)
- net at J2.13 (Pin_13), U12.9 (SA), U17.2: now also RN2.5 (R4)
- net at J2.14 (Pin_14), U12.14 (SB), U17.4: now also RN2.6 (R5)
- net at J2.15 (Pin_15), U14.1, U17.6: now also RN2.7 (R6)
- net at J2.16 (Pin_16), U17.8: now also Q1.3 (C), RN2.8 (R7)
- net at J2.17 (Pin_17), U17.10: now also RN2.9 (R8)
- net at J2.18 (Pin_18), U17.12: now also RN2.10 (R9)
- net at R16.2, RV1.1: no longer Q1.2 (B), RV1.2
- new net: C8.1, U1.4 (V-), U4.4 (V-), U5.7 (VSS), U6.4 (V-)
- new net: Q1.2 (B), RV1.2
Other:
- note added: "ANALOG\nOFF BOARD\nOPTION\nFOR STM32\nDACs/COMPs"
- note added: "TEST\nTHIS \nVALUE"
- note removed: "PIN 20 MUST BE 5V \nTOLERANT INPUT"
- note removed: "or 15k"
- moved on the sheet: C1, C2, C3, C7, Q1, R16, R21, RV1, TP11, U15G, U16G, U17G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

Commit message: Updates.
Parts:
- removed C13, C14, C17, C18: 100p, symbol Device:C
- removed C4: .1u, symbol Device:C
- removed R3: 1k, symbol Device:R
- removed R30: 100k, symbol Device:R
- removed TP6: TestPoint, TestPoint:TestPoint_THTPad_2.5x2.5mm_Drill1.2mm, symbol Connector:TestPoint
- removed unit 2 of U1
- removed unit 3 of U1
- added U18: MCP4901, symbol Analog_DAC:MCP4901
- added U19: MAX4544, Package_DIP:DIP-8_W7.62mm_Socket, symbol Analog_Switch:MAX4544
- R2: value 1k -> 2.2k
- R22, R23: value 33k -> 11k
- R24, R25: value 33k -> 15k
- U1: value LM2904 -> OPA347; symbol Amplifier_Operational:LM2904 -> Amplifier_Operational:OPA340P
- U6: value LF412CP -> MCP6292
Connections:
- net +5V: now also Q1.3 (C), U1.7 (V+), U18.1 (Vdd), U18.6 (Vref), U19.8 (V+)
- net GND: now also R2.1, U1.4 (V-), U18.5 (~LDAC), U18.7 (Vss), U19.3 (NC), U19.4 (GND); no longer RV1.3, U14.4, U14.5
- net at J1.2 (Pin_2), TP2.1, U4.1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: now also R5.2; no longer R2.2
- net at J1.1 (Pin_1), R11.2, R4.2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: now also U1.6; no longer U1.1
- net at J1.3 (Pin_3), TP3.1, U4.6 (-)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: now also R7.2
- net at U5.3: now also R5.1; no longer R5.2
- net at U5.4: now also C11.2, U5.2, U6.2 (-); no longer R2.1
- net at U5.8: now also C12.2, U5.10, U6.6 (-)
- net at U5.9: now also R7.1; no longer R7.2
- net at C11.1, J1.4 (Pin_4), R8.2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: now also C12.1, J1.5 (Pin_5), R10.2, TP5.1, U5.1, U5.11, U6.7, U9.9 (+); no longer U5.2
- net at J2.9 (Pin_9), RN1.10 (R9), U10.4 (SCK)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: now also U18.3 (SCK)
- net at J2.10 (Pin_10), RN2.2 (R1), U10.5 (SDI)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: now also U18.4 (SDI)
- net at J2.16 (Pin_16), RN2.8 (R7), U17.8: now also U14.4; no longer Q1.3 (C)
- net at J2.17 (Pin_17), RN2.9 (R8), U17.10: now also U18.2 (~CS)
- net at U14.6: now also U19.7 (IN)
- net at U14.3: now also U14.5; no longer R16.1
- new net: U18.8 (Vout), U19.1 (NO)
- new net: R2.2, RV1.3
- new net: R16.1, U19.2 (COM)
Other:
- note added: "COEFFICIENT BUFFERS"
- note added: "COEFFICIENT DACS"
- note added: "INSTALL EITHER:\n- DAC U18 & MAX4544 (Z analog control)\n- or leave both uninstalled \n and jumper IN and COM on MAX4544 footprint"
- note added: "Integrator amp\nshould be rail-to-rail output"
- note removed: "COEFFICIENT DAC BUFFERS"
- note removed: "TEST\nTHIS \nVALUE"
- note removed: "TODO: Change to \nOPA705 or OPA347"
- note removed: "TODO:\nCheck if \nthis resistor \nactually helps"
- moved on the sheet: Q1, R16, R21, R5, R7, RV1, TP11, U5A, U5B, U5C, U5D, U9C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

Commit message: Replace Yamaha DACs with MCP4922 for coefficients.
Parts:
- removed C5, C6: .1u, symbol Device:C
- removed R28, R29: 100k, symbol Device:R
- removed U2, U3: Y3014B, Package_DIP:DIP-8_W7.62mm_Socket, symbol Analog_DAC:Y3014B
- removed unit 1 of U4
- removed unit 2 of U4
- added U?: MCP4922, symbol Analog_DAC:MCP4922
- R4, R6: value 4.7k -> 10k
- R5, R7: value 4.7k -> 15k
Connections:
- wire segments 530 -> 499
Other:
- note added: "HOLD will unblank Z when raised \n(to ensure there is no software delay \nbetween start of integration & unblanking)"
- note added: "LIMIT_LOW: Invert sense\nof comparator output \n(according to direction\nof integration)"
- note added: "Select R17 and R18 to be as close as possible\nand R24 to be as close as possible to (15/33)*that value"
- note added: "Select R19 and R20 to be as close as possible\nand R25 to be as close as possible to (15/33)*that value"
- note added: "Select R4 and R6 to be \nas close as possible\nSelect C11 and C12 to be \nas close as possible"
- note added: "Select all four resistors\nto be as close as possible"
- note removed: "COEFFICIENT BUFFERS"
- note removed: "When HIGH this signal\nwill invert the comparator\noutput"
- moved on the sheet: C1, C10, C11, C12, C15, C16, C19, C2, C20, C3, C7, C8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

Commit message: Snapshot of work in progress pcb.
Parts:
- removed C3: 1u, symbol Device:C
- removed J1: Conn_01x06_Female, symbol Connector:Conn_01x06_Female
- removed J2, J3: Conn_01x20_Female, symbol Connector:Conn_01x20_Female
- removed J4: Conn_01x04_Male, symbol Connector:Conn_01x04_Male
- removed R2: 2.2k, symbol Device:R
- removed R31, R32: 100k, symbol Device:R
- removed RN1: R_Network09_US, Resistor_THT:R_Array_SIP10, symbol Device:R_Network09_US
- removed U1: OPA347, symbol Amplifier_Operational:OPA340P
- removed U15: 74LS07, symbol 74xx:74LS07
- removed U18: MCP4901, symbol Analog_DAC:MCP4901
- removed U4: MCP6292, symbol Amplifier_Operational:LM2904
- added J1: ARDUINO POWER 3.3V, Connector_PinHeader_2.54mm:PinHeader_1x06_P2.54mm_Vertical, symbol Connector_Generic:Conn_01x06
- added J10: ARDUINO J1, Connector_PinHeader_2.54mm:PinHeader_1x08_P2.54mm_Vertical, symbol Connector_Generic:Conn_01x08
- added J11: Conn_01x08, Connector_PinHeader_2.54mm:PinHeader_1x08_P2.54mm_Vertical, symbol Connector_Generic:Conn_01x08
- added J2: ARDUINO J3 3.3V, Connector_PinHeader_2.54mm:PinHeader_1x08_P2.54mm_Vertical, symbol Connector_Generic:Conn_01x08
- added J3: ARDUINO J2 3.3V, Connector_PinHeader_2.54mm:PinHeader_1x06_P2.54mm_Vertical, symbol Connector_Generic:Conn_01x06
- added J5: ARDUINO J1 3.3V, Connector_PinHeader_2.54mm:PinHeader_1x08_P2.54mm_Vertical, symbol Connector_Generic:Conn_01x08
- added J6: Conn_01x03, Connector_Molex:Molex_KK-396_A-41791-0003_1x03_P3.96mm_Vertical, symbol Connector_Generic:Conn_01x03
- added J7: ARDUINO POWER, Connector_PinHeader_2.54mm:PinHeader_1x06_P2.54mm_Vertical, symbol Connector_Generic:Conn_01x06
- added J8: ARDUINO J3, Connector_PinHeader_2.54mm:PinHeader_1x08_P2.54mm_Vertical, symbol Connector_Generic:Conn_01x08
- added J9: ARDUINO J2, Connector_PinHeader_2.54mm:PinHeader_1x06_P2.54mm_Vertical, symbol Connector_Generic:Conn_01x06
- added R28, R29, R30, R33: 10k, Resistor_THT:R_Axial_DIN0207_L6.3mm_D2.5mm_P10.16mm_Horizontal, symbol Device:R
- added R3: 4.7k, Resistor_THT:R_Axial_DIN0207_L6.3mm_D2.5mm_P10.16mm_Horizontal, symbol Device:R
- added R34, R35: 47, Resistor_THT:R_Axial_DIN0207_L6.3mm_D2.5mm_P10.16mm_Horizontal, symbol Device:R
- added TP17, TP18, TP19, TP20, TP21, TP22, TP6: TestPoint, TestPoint:TestPoint_THTPad_2.5x2.5mm_Drill1.2mm, symbol Connector:TestPoint
- C1, C10, C15, C16, C19, C2, C20, C7, C8, C9: footprint (none) -> Capacitor_THT:C_Disc_D5.0mm_W2.5mm_P2.50mm
- C11, C12: footprint (none) -> Capacitor_THT:C_Rect_L7.0mm_W2.5mm_P5.00mm
- Q1: footprint Package_TO_SOT_THT:TO-92_Inline -> Package_TO_SOT_THT:TO-92_HandSolder
- R1, R10, R11, R12, R13, R14, R15, R16, R17, R18, R19, R20, R21, R22, R23, R24, R25, R26, R27, R4, R5, R6, R7, R8, R9: footprint (none) -> Resistor_THT:R_Axial_DIN0207_L6.3mm_D2.5mm_P10.16mm_Horizontal
- RV1: footprint (none) -> Potentiometer_THT:Potentiometer_TT_P0915N
- U1: renamed from U?; footprint (none) -> Package_DIP:DIP-14_W7.62mm_Socket
- U10, U11, U14, U16, U17, U5, U9: footprint (none) -> Package_DIP:DIP-14_W7.62mm_Socket
- U12: footprint (none) -> Package_DIP:DIP-16_W7.62mm_Socket
- U13: footprint (none) -> Package_TO_SOT_THT:TO-92_HandSolder
- U6, U7, U8: footprint (none) -> Package_DIP:DIP-8_W7.62mm_Socket
- XOUT1, YOUT1, ZOUT1: footprint (none) -> Connector_Coaxial:BNC_TEConnectivity_1478204_Vertical
Connections:
- net labels added: +3.3V
- wire segments 499 -> 483
Other:
- note added: "ANALOG OFF BOARD\nOPTION FOR STM32\nDACs/COMPs"
- note added: "COMP: output of \nselected comparator, \nmay need inversion"
- note added: "Divide the\nSTOP signal\nto approx 3.4V"
- note added: "LIMIT_LOW: Invert sense of comparator output \n(according to direction of integration)"
- note added: "STOP signal to MCU\n"
- note added: "The analog switches and DACs are 5V controlled, so we need\nbuffers and pullups to level-shift when 3.3V control is used"
- note added: "Z = COMPARATOR OUT ^ LIMIT_LOW ^ HOLD ^ Z_BLANK\n\n& the master switch signal Z_ENABLE uses U19\nto switch Z to 0V regardless of the logic output.\n\nWhile a line is being drawn (integrators running): \nCOMPARATOR SELECT lines are set according to \nwhich should set COMP OUT;\nHOLD is HIGH; Z_BLANK is low (don’t invert);\nresulting in Z output HIGH.\nWhen integrator limit is reached, COMP OUT fli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"
- note added: "Z CONTROL LOGIC\n"
- note added: "Z_BLANK switches Z when HOLD is low\n(integrators not running)"
- note removed: "3.3V DIGITAL INPUTS\n(PIN 20 IS 5V OUTPUT)"
- note removed: "ANALOG\nOFF BOARD\nOPTION\nFOR STM32\nDACs/COMPs"
- note removed: "INSTALL EITHER:\n- DAC U18 & MAX4544 (Z analog control)\n- or leave both uninstalled \n and jumper IN and COM on MAX4544 footprint"
- note removed: "LIMIT_LOW: Invert sense\nof comparator output \n(according to direction\nof integration)"
- moved on the sheet: R1, RN2, TP4, TP5, U13, U14D, U16A, U16B, U16C, U16D, U16E, U16F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

Commit message: Snapshot of work in progress pcb.
Parts:
- removed C8: 1u, Capacitor_THT:C_Disc_D5.0mm_W2.5mm_P2.50mm, symbol Device:C
- added C3, C4, C5: 1u, Capacitor_THT:C_Disc_D5.0mm_W2.5mm_P2.50mm, symbol Device:C
Connections:
- net +5V: now also C3.2, C4.2, C5.2
- net -5V: no longer R21.1
- net GND: now also R21.1, U5.7 (VSS), C3.1, C4.1, C5.1
- net at C10.1, U6.4 (V-): no longer U5.7 (VSS)
Changed lines of the file:
@@
 $EndComp
-Wire Wire Line
-	8300 1275 8300 1375
-Connection ~ 8300 1275
-Wire Wire Line
-	8675 1275 8675 1450
-Wire Wire Line
-	8300 1275 8675 1275
-Wire Wire Line
-	8300 1825 9025 1825
-Wire Wire Line
-	8300 1675 8300 1825
-Wire Wire Line
-	8300 1200 8300 1275
 Wire Wire Line
 	8300 725  8300 900
@@
 L power:GND #PWR014
 U 1 1 62992F3E
-P 8675 1450
-F 0 "#PWR014" H 8675 1200 50  0001 C CNN
-F 1 "GND" H 8680 1277 50  0000 C CNN
-F 2 "" H 8675 1450 50  0001 C CNN
-F 3 "" H 8675 1450 50  0001 C CNN
-	1    8675 1450
-	1    0    0    -1
-$EndComp
-$Comp
-L Device:C C8
-U 1 1 62991005
-P 8300 1525
-F 0 "C8" V 8048 1525 50  0000 C CNN
-F 1 "1u" V 8139 1525 50  0000 C CNN
-F 2 "Capacitor_THT:C_Disc_D5.0mm_W2.5mm_P2.50mm" H 8338 1375 50  0001 C CNN
-F 3 "~" H 8300 1525 50  0001 C CNN
-	1    8300 1525
-	-1   0    0    1
+P 8300 1925
+F 0 "#PWR014" H 8300 1675 50  0001 C CNN
+F 1 "GND" H 8305 1752 50  0000 C CNN
+F 2 "" H 8300 1925 50  0001 C CNN
+F 3 "" H 8300 1925 50  0001 C CNN
+	1    8300 1925
+	1    0    0    -1
 $EndComp
 Wire Wire Line
 	9025 725  9550 725
-Wire Wire Line
-	9025 1825 9550 1825
 $Comp
 L Device:C C7
@@
 	-1   0    0    1
 $EndComp
-Connection ~ 9025 1825
 Wire Wire Line
 	10300 1825 10300 1775
@@
 	11550 10150 11550 10250
 $Comp
-L power:-5V #PWR022
-U 1 1 62C16B97
-P 11550 10250
-F 0 "#PWR022" H 11550 10350 50  0001 C CNN
-F 1 "-5V" H 11565 10423 50  0000 C CNN
-F 2 "" H 11550 10250 50  0001 C CNN
-F 3 "" H 11550 10250 50  0001 C CNN
-	1    11550 10250
-	-1   0    0    1
-$EndComp
-$Comp
 L Device:R R21
 U 1 1 62C16599
@@
 Wire Wire Line
 	9550 725  10300 725
-Connection ~ 9550 1825
 Wire Wire Line
 	9550 1825 10300 1825
@@
 Connection ~ 8000 5700
 Wire Wire Line
-	8000 5700 9225 5700
-Wire Wire Line
 	6975 2975 6975 4875
 Wire Wire Line
@@
 Wire Wire Line
 	10975 9675 10975 10250
+$Comp
+L Device:C C3
+U 1 1 62586135
+P 4550 4100
+F 0 "C3" V 4298 4100 50  0000 C CNN
+F 1 "1u" V 4389 4100 50  0000 C CNN
+F 2 "Capacitor_THT:C_Disc_D5.0mm_W2.5mm_P2.50mm" H 4588 3950 50  0001 C CNN
+F 3 "~" H 4550 4100 50  0001 C CNN
+	1    4550 4100
+	-1   0    0    1
+$EndComp
+$Comp
+L Device:C C4
+U 1 1 62586CE9
+P 4550 5550
+F 0 "C4" V 4298 5550 50  0000 C CNN
+F 1 "1u" V 4389 5550 50  0000 C CNN
+F 2 "Capacitor_THT:C_Disc_D5.0mm_W2.5mm_P2.50mm" H 4588 5400 50  0001 C CNN
+F 3 "~" H 4550 5550 50  0001 C CNN
+	1    4550 5550
+	-1   0    0    1
+$EndComp
+Wire Wire Line
+	8000 5700 9225 5700
+$Comp
+L Device:C C5
+U 1 1 62589EBF
+P 8350 5950
+F 0 "C5" V 8098 5950 50  0000 C CNN
+F 1 "1u" V 8189 5950 50  0000 C CNN
+F 2 "Capacitor_THT:C_Disc_D5.0mm_W2.5mm_P2.50mm" H 8388 5800 50  0001 C CNN
+F 3 "~" H 8350 5950 50  0001 C CNN
+	1    8350 5950
+	-1   0    0    1
+$EndComp
+Wire Wire Line
+	4550 3750 4550 3950
+Connection ~ 4550 3750
+Wire Wire Line
+	5125 5350 4550 5350
+Wire Wire Line
+	4550 5350 4550 5400
+Connection ~ 5125 5350
+Wire Wire Line
+	7125 5350 8350 5350
+Wire Wire Line
+	8350 5350 8350 5800
+Connection ~ 7125 5350
+$Comp
+L power:GND #PWR0113
+U 1 1 626711F0
+P 4550 5700
+F 0 "#PWR0113" H 4550 5450 50  0001 C CNN
+F 1 "GND" H 4555 5527 50  0000 C CNN
+F 2 "" H 4550 5700 50  0001 C CNN
+F 3 "" H 4550 5700 50  0001 C CNN
+	1    4550 5700
+	1    0    0    -1
+$EndComp
+$Comp
+L power:GND #PWR0114
+U 1 1 62671E41
+P 8350 6100
+F 0 "#PWR0114" H 8350 5850 50  0001 C CNN
+F 1 "GND" H 8355 5927 50  0000 C CNN
+F 2 "" H 8350 6100 50  0001 C CNN
+F 3 "" H 8350 6100 50  0001 C CNN
+	1    8350 6100
+	1    0    0    -1
+$EndComp
+$Comp
+L power:GND #PWR0115
+U 1 1 62672390
+P 4550 4250
+F 0 "#PWR0115" H 4550 4000 50  0001 C CNN
+F 1 "GND" H 4555 4077 50  0000 C CNN
+F 2 "" H 4550 4250 50  0001 C CNN
+F 3 "" H 4550 4250 50  0001 C CNN
+	1    4550 4250
+	1    0    0    -1
+$EndComp
+Connection ~ 8300 1825
+Wire Wire Line
+	8300 1200 8300 1825
+Wire Wire Line
+	8300 1925 8300 1825
+Wire Wire Line
+	8300 1825 9025 1825
+$Comp
+L power:GND #PWR?
+U 1 1 627D9B7D
+P 11550 10250
+F 0 "#PWR?" H 11550 10000 50  0001 C CNN
+F 1 "GND" H 11555 10077 50  0000 C CNN
+F 2 "" H 11550 10250 50  0001 C CNN
+F 3 "" H 11550 10250 50  0001 C CNN
+	1    11550 10250
+	1    0    0    -1
+$EndComp
 $EndSCHEMATC
