File: vector_gen/vector_gen.sch (KiCad schematic (older format))
At the start: 88 parts, among them J1 ARDUINO POWER 3.3V, J10 ARDUINO J1, J11 Conn_01x08, J2 ARDUINO J3 3.3V, J3 ARDUINO J2 3.3V, J4 Conn_01x02_Female, J5 ARDUINO J1 3.3V, J6 Conn_01x03, J7 ARDUINO POWER, J8 ARDUINO J3, J9 ARDUINO J2, Q1 2N3904, U1 MCP4922, U10 MCP4922, U11 MCP4922, U12 4019, U13 LM336, U14 74HC86, U16 74LS07, U17 74LS07, U19 MAX4544, U5 4066, U6 MCP6292, U7 TL072IP, U8 TL072IP, U9 LM319

Commit message: Rerrange layout
Parts:
- added H1, H2, H3, H4: MountingHole, MountingHole:MountingHole_3.2mm_M3, symbol Mechanical:MountingHole
Changed lines of the file:
@@
 Wire Wire Line
 	7500 4975 8000 4975
+$Comp
+L Mechanical:MountingHole H1
+U 1 1 626931D6
+P 13550 1375
+F 0 "H1" H 13650 1421 50  0000 L CNN
+F 1 "MountingHole" H 13650 1330 50  0000 L CNN
+F 2 "MountingHole:MountingHole_3.2mm_M3" H 13550 1375 50  0001 C CNN
+F 3 "~" H 13550 1375 50  0001 C CNN
+	1    13550 1375
+	1    0    0    -1
+$EndComp
+$Comp
+L Mechanical:MountingHole H2
+U 1 1 62693475
+P 13550 1675
+F 0 "H2" H 13650 1721 50  0000 L CNN
+F 1 "MountingHole" H 13650 1630 50  0000 L CNN
+F 2 "MountingHole:MountingHole_3.2mm_M3" H 13550 1675 50  0001 C CNN
+F 3 "~" H 13550 1675 50  0001 C CNN
+	1    13550 1675
+	1    0    0    -1
+$EndComp
+$Comp
+L Mechanical:MountingHole H3
+U 1 1 6269382A
+P 14400 1375
+F 0 "H3" H 14500 1421 50  0000 L CNN
+F 1 "MountingHole" H 14500 1330 50  0000 L CNN
+F 2 "MountingHole:MountingHole_3.2mm_M3" H 14400 1375 50  0001 C CNN
+F 3 "~" H 14400 1375 50  0001 C CNN
+	1    14400 1375
+	1    0    0    -1
+$EndComp
+$Comp
+L Mechanical:MountingHole H4
+U 1 1 62693BCB
+P 14400 1675
+F 0 "H4" H 14500 1721 50  0000 L CNN
+F 1 "MountingHole" H 14500 1630 50  0000 L CNN
+F 2 "MountingHole:MountingHole_3.2mm_M3" H 14400 1675 50  0001 C CNN
+F 3 "~" H 14400 1675 50  0001 C CNN
+	1    14400 1675
+	1    0    0    -1
+$EndComp
 $EndSCHEMATC

Commit message: Ground plane done?
Parts:
- added D1: LED, LED_THT:LED_D3.0mm, symbol Device:LED
- added R2: 330, Resistor_THT:R_Axial_DIN0207_L6.3mm_D2.5mm_P10.16mm_Horizontal, symbol Device:R
Connections:
- net +5V: now also D1.2 (A)
- net GND: now also R2.2
- new net: D1.1 (K), R2.1
Other:
- note added: "LED voltage drop (red) 1.7V\n10mA = (5-1.7)/R \nR = 3.3/0.01 = 330Ω\n"
Changed lines of the file:
@@
 	1250 2275 1250 2025
 Wire Wire Line
-	1000 2375 1550 2375
+	1000 2375 1375 2375
 Wire Wire Line
 	1550 2375 1550 2400
@@
 	1    0    0    -1
 $EndComp
+$Comp
+L Device:LED D1
+U 1 1 626BE9D5
+P 1775 2050
+F 0 "D1" V 1814 1932 50  0000 R CNN
+F 1 "LED" V 1723 1932 50  0000 R CNN
+F 2 "LED_THT:LED_D3.0mm" H 1775 2050 50  0001 C CNN
+F 3 "~" H 1775 2050 50  0001 C CNN
+	1    1775 2050
+	0    -1   -1   0
+$EndComp
+$Comp
+L Device:R R2
+U 1 1 626C1DE2
+P 1775 2475
+F 0 "R2" H 1845 2521 50  0000 L CNN
+F 1 "330" H 1845 2430 50  0000 L CNN
+F 2 "Resistor_THT:R_Axial_DIN0207_L6.3mm_D2.5mm_P10.16mm_Horizontal" V 1705 2475 50  0001 C CNN
+F 3 "~" H 1775 2475 50  0001 C CNN
+	1    1775 2475
+	1    0    0    -1
+$EndComp
+Text Notes 800  1425 0    50   ~ 0
+LED voltage drop (red) 1.7V\n10mA = (5-1.7)/R \nR = 3.3/0.01 = 330Ω\n
+Wire Wire Line
+	1775 2200 1775 2325
+Wire Wire Line
+	1775 2625 1775 2725
+Wire Wire Line
+	1775 2725 1375 2725
+Wire Wire Line
+	1250 2275 1375 2275
+Wire Wire Line
+	1375 2275 1375 1900
+Wire Wire Line
+	1375 1900 1775 1900
+Connection ~ 1250 2275
+Connection ~ 1375 2375
+Wire Wire Line
+	1375 2375 1550 2375
+Wire Wire Line
+	1375 2375 1375 2725
 $EndSCHEMATC

Commit message: Add fill to front copper and suggestions from joe_z.
Parts:
- removed R12, R13, R14, R15: 33k, Resistor_THT:R_Axial_DIN0207_L6.3mm_D2.5mm_P10.16mm_Horizontal, symbol Device:R
- removed U7: TL072IP, Package_DIP:DIP-8_W7.62mm_Socket, symbol Amplifier_Operational:TL072
- added C13, C14, C17, C18: .1u, Capacitor_THT:C_Disc_D5.0mm_W2.5mm_P2.50mm, symbol Device:C
- added C6, C8: 100u, Capacitor_THT:C_Radial_D6.3mm_H7.0mm_P2.50mm, symbol Device:CP
- R22, R23: value 11k -> 15k
Connections:
- net +5V: now also C6.1
- net -5V: now also C8.2
- net GND: now also C13.1, C14.1, C17.1, C18.1, C6.2, C8.1
- net at J11.7 (Pin_7), J2.8 (Pin_8), J8.8 (Pin_8)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: now also R10.2, R8.2
- net at C11.1, TP4.1, U5.1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: now also R17.2; no longer R8.2
- net at R4.1, U6.3 (+): now also C13.2
- net at R6.1, U6.5 (+): now also C14.2
- net at C12.1, TP5.1, U5.11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: now also R19.2; no longer R10.2
- net at R9.1: now also R22.2, R8.1, U8.3 (+), C17.2
- net at R10.1: now also R11.1, R23.2, U8.5 (+), C18.2
Other:
- note removed: "INTEGRATOR UNBIAS"
- note removed: "Integrator maximum slew\n1.25/RC = 0.027 V/µs (check this, doesn’t seem right)"
- note removed: "Select R17 and R18 to be as close as possible\nand R24 to be as close as possible to (15/33)*that value"
- note removed: "Select R19 and R20 to be as close as possible\nand R25 to be as close as possible to (15/33)*that value"
- note removed: "Select all four resistors\nto be as close as possible"
- moved on the sheet: J6, R10, R11, R22, R8, R9

Commit message: Updated.
Parts:
- added C21, C22: 1u, Capacitor_THT:C_Disc_D5.0mm_W2.5mm_P2.50mm, symbol Device:C
- added R12, R13: 100k? to be determined, Resistor_THT:R_Axial_DIN0207_L6.3mm_D2.5mm_P10.16mm_Horizontal, symbol Device:R
Connections:
- net +5V: now also C21.2
- net -5V: now also C22.1
- net GND: now also C21.1, C22.2
- net at C11.1, R17.2, TP4.1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: now also R12.2
- net at C12.1, R19.2, TP5.1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: now also R13.2
- net at R26.1, U12.6 (A0), U9.12: now also R12.1
- net at R27.1, U12.7 (B0), U9.7: now also R13.1
Other:
- moved on the sheet: C1, C10, C11, C12, C13, C14, C15, C16, C17, C18, C19, C2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

Commit message: Some important corrections. OSHpark candidate?
Parts:
- added J12: Conn_01x02, Connector_PinSocket_2.54mm:PinSocket_1x02_P2.54mm_Vertical, symbol Connector_Generic:Conn_01x02
- added PB0, PC4, PC5: TestPoint, TestPoint:TestPoint_THTPad_2.5x2.5mm_Drill1.2mm, symbol Connector:TestPoint
- renumbered TP16 to STOP1, TP1 to VREF2.5, TP12 to X1, TP2 to XCOEFF1, TP4 to XINTEG1, TP14 to XLIMIT1, TP13 to Y1, TP3 to YCOEFF1, TP5 to YINTEG1, TP15 to YLIMIT1, TP11 to Z1
Connections:
- net +3V3: now also J1.5 (Pin_5); no longer J1.2 (Pin_2)
- net GND: now also J1.2 (Pin_2), J1.3 (Pin_3), J7.2 (Pin_2), J7.3 (Pin_3); no longer J1.4 (Pin_4), J1.5 (Pin_5), J7.4 (Pin_4), J7.5 (Pin_5)
- net at J2.1 (Pin_1), J8.1 (Pin_1): now also PB0.1
- net at J8.3 (Pin_3): no longer J2.3 (Pin_3)
- net at J8.5 (Pin_5): no longer J2.5 (Pin_5)
- net at J3.5 (Pin_5), J9.5 (Pin_5): now also PC4.1
- net at J3.6 (Pin_6), J9.6 (Pin_6): now also PC5.1
- net at J10.1 (Pin_1), J5.1 (Pin_1): now also J12.2 (Pin_2)
- net at J10.2 (Pin_2), J5.2 (Pin_2): now also J12.1 (Pin_1)
Changed lines of the file:
@@
 Wire Wire Line
 	11425 6725 10925 6725
-Wire Wire Line
-	10925 6725 10350 6725
 Connection ~ 10925 6725
 Wire Wire Line
@@
 $EndComp
 $Comp
-L Connector:TestPoint TP11
+L Connector:TestPoint Z1
 U 1 1 6228F9FB
 P 16450 10275
-F 0 "TP11" H 16508 10393 50  0000 L CNN
+F 0 "Z1" H 16508 10393 50  0000 L CNN
 F 1 "TestPoint" H 16508 10302 50  0000 L CNN
 F 2 "TestPoint:TestPoint_THTPad_2.5x2.5mm_Drill1.2mm" H 16650 10275 50  0001 C CNN
@@
 $EndComp
 Connection ~ 19675 7800
-$Comp
-L Connector:TestPoint TP16
-U 1 1 6219D120
-P 19675 7800
-F 0 "TP16" H 19733 7918 50  0000 L CNN
-F 1 "TestPoint" H 19733 7827 50  0000 L CNN
-F 2 "TestPoint:TestPoint_THTPad_2.5x2.5mm_Drill1.2mm" H 19875 7800 50  0001 C CNN
-F 3 "~" H 19875 7800 50  0001 C CNN
-	1    19675 7800
-	1    0    0    -1
-$EndComp
 Wire Wire Line
 	17050 8850 17325 8850
 Connection ~ 17050 8850
 $Comp
-L Connector:TestPoint TP15
+L Connector:TestPoint YLIMIT1
 U 1 1 6219C247
 P 17050 8850
-F 0 "TP15" H 17108 8968 50  0000 L CNN
+F 0 "YLIMIT1" H 17108 8968 50  0000 L CNN
 F 1 "TestPoint" H 17108 8877 50  0000 L CNN
 F 2 "TestPoint:TestPoint_THTPad_2.5x2.5mm_Drill1.2mm" H 17250 8850 50  0001 C CNN
@@
 Connection ~ 17050 8175
 $Comp
-L Connector:TestPoint TP14
+L Connector:TestPoint XLIMIT1
 U 1 1 6219BC30
 P 17050 8175
-F 0 "TP14" H 17108 8293 50  0000 L CNN
+F 0 "XLIMIT1" H 17108 8293 50  0000 L CNN
 F 1 "TestPoint" H 17108 8202 50  0000 L CNN
 F 2 "TestPoint:TestPoint_THTPad_2.5x2.5mm_Drill1.2mm" H 17250 8175 50  0001 C CNN
@@
 $EndComp
 $Comp
-L Connector:TestPoint TP5
+L Connector:TestPoint YINTEG1
 U 1 1 6219AA65
 P 14400 6300
-F 0 "TP5" H 14458 6418 50  0000 L CNN
+F 0 "YINTEG1" H 14458 6418 50  0000 L CNN
 F 1 "TestPoint" H 14458 6327 50  0000 L CNN
 F 2 "TestPoint:TestPoint_THTPad_2.5x2.5mm_Drill1.2mm" H 14600 6300 50  0001 C CNN
@@
 $EndComp
 $Comp
-L Connector:TestPoint TP4
+L Connector:TestPoint XINTEG1
 U 1 1 6219A424
 P 14325 4875
-F 0 "TP4" H 14383 4993 50  0000 L CNN
+F 0 "XINTEG1" H 14383 4993 50  0000 L CNN
 F 1 "TestPoint" H 14383 4902 50  0000 L CNN
 F 2 "TestPoint:TestPoint_THTPad_2.5x2.5mm_Drill1.2mm" H 14525 4875 50  0001 C CNN
@@
 $EndComp
 $Comp
-L Connector:TestPoint TP13
+L Connector:TestPoint Y1
 U 1 1 62199DA2
 P 17050 6300
-F 0 "TP13" H 17108 6418 50  0000 L CNN
+F 0 "Y1" H 17108 6418 50  0000 L CNN
 F 1 "TestPoint" H 17108 6327 50  0000 L CNN
 F 2 "TestPoint:TestPoint_THTPad_2.5x2.5mm_Drill1.2mm" H 17250 6300 50  0001 C CNN
@@
 $EndComp
 $Comp
-L Connector:TestPoint TP12
+L Connector:TestPoint X1
 U 1 1 62199961
 P 17050 4875
-F 0 "TP12" H 17108 4993 50  0000 L CNN
+F 0 "X1" H 17108 4993 50  0000 L CNN
 F 1 "TestPoint" H 17108 4902 50  0000 L CNN
 F 2 "TestPoint:TestPoint_THTPad_2.5x2.5mm_Drill1.2mm" H 17250 4875 50  0001 C CNN
@@
 $EndComp
 $Comp
-L Connector:TestPoint TP3
+L Connector:TestPoint YCOEFF1
 U 1 1 621987EB
 P 11575 5525
-F 0 "TP3" H 11633 5643 50  0000 L CNN
+F 0 "YCOEFF1" H 11633 5643 50  0000 L CNN
 F 1 "TestPoint" H 11633 5552 50  0000 L CNN
 F 2 "TestPoint:TestPoint_THTPad_2.5x2.5mm_Drill1.2mm" H 11775 5525 50  0001 C CNN
@@
 $EndComp
 $Comp
-L Connector:TestPoint TP2
+L Connector:TestPoint XCOEFF1
 U 1 1 62198169
 P 11575 4975
-F 0 "TP2" H 11633 5093 50  0000 L CNN
+F 0 "XCOEFF1" H 11633 5093 50  0000 L CNN
 F 1 "TestPoint" H 11633 5002 50  0000 L CNN
 F 2 "TestPoint:TestPoint_THTPad_2.5x2.5mm_Drill1.2mm" H 11775 4975 50  0001 C CNN
@@
 $EndComp
 $Comp
-L Connector:TestPoint TP1
+L Connector:TestPoint VREF2.5
 U 1 1 6214E9C9
 P 10375 3675
-F 0 "TP1" H 10433 3793 50  0000 L CNN
+F 0 "VREF2.5" H 10433 3793 50  0000 L CNN
 F 1 "TestPoint" H 10433 3702 50  0000 L CNN
 F 2 "TestPoint:TestPoint_THTPad_2.5x2.5mm_Drill1.2mm" H 10575 3675 50  0001 C CNN
@@
 Wire Wire Line
 	10925 7475 10925 8075
-Wire Wire Line
-	10350 6725 9925 6725
-Connection ~ 10350 6725
-Wire Wire Line
-	10350 6500 10350 6725
 Text Notes 13650 7725 0    79   ~ 0
 INTEGRATORS\n
@@
 L power:+5V #PWR09
 U 1 1 6202B606
-P 10350 6500
-F 0 "#PWR09" H 10350 6350 50  0001 C CNN
-F 1 "+5V" H 10365 6673 50  0000 C CNN
-F 2 "" H 10350 6500 50  0001 C CNN
-F 3 "" H 10350 6500 50  0001 C CNN
-	1    10350 6500
+P 8850 6475
+F 0 "#PWR09" H 8850 6325 50  0001 C CNN
+F 1 "+5V" H 8865 6648 50  0000 C CNN
+F 2 "" H 8850 6475 50  0001 C CNN
+F 3 "" H 8850 6475 50  0001 C CNN
+	1    8850 6475
 	1    0    0    -1
 $EndComp
@@
 	-1   0    0    1
 $EndComp
-Wire Wire Line
-	5300 5925 5525 5925
-Wire Wire Line
-	5525 5925 5525 6675
-$Comp
-L power:GND #PWR0102
-U 1 1 62BF8DD0
-P 5525 6675
-F 0 "#PWR0102" H 5525 6425 50  0001 C CNN
-F 1 "GND" H 5530 6502 50  0000 C CNN
-F 2 "" H 5525 6675 50  0001 C CNN
-F 3 "" H 5525 6675 50  0001 C CNN
-	1    5525 6675
-	1    0    0    -1
-$EndComp
 Connection ~ 9300 6025
 Wire Wire Line
@@
 	3425 6850 3425 6900
 Wire Wire Line
-	1675 6125 5300 6125
-Wire Wire Line
-	1675 6325 5300 6325
-Wire Wire Line
-	1675 6525 5300 6525
-Wire Wire Line
 	1675 7025 5300 7025
 Wire Wire Line
@@
 	1675 8500 5300 8500
 Wire Wire Line
-	1675 8600 5300 8600
-Wire Wire Line
 	8500 7900 8500 9275
 Wire Wire Line
@@
 Wire Wire Line
 	7625 2500 7625 4275
-Connection ~ 5525 4925
-Wire Wire Line
-	5525 4825 5525 4925
-Wire Wire Line
-	5300 4825 5525 4825
-Wire Wire Line
-	5300 4925 5525 4925
-Wire Wire Line
-	5525 4925 5525 5350
 $Comp
 L power:GND #PWR0107
@@
 	-1   0    0    1
 $EndComp
-Connection ~ 1900 4925
-Wire Wire Line
-	1900 4825 1900 4925
-Wire Wire Line
-	1675 4825 1900 4825
-Wire Wire Line
-	1675 4925 1900 4925
-Wire Wire Line
-	1900 4925 1900 5350
 $Comp
 L power:GND #PWR0108
@@
 $EndComp
 Wire Wire Line
-	2350 4425 2350 5125
-Wire Wire Line
-	2350 5125 1675 5125
+	2350 4425 2350 4825
 Wire Wire Line
 	8375 10450 12375 10450
@@
 Wire Wire Line
 	20150 8025 20150 8700
+Wire Wire Line
+	9925 6725 10925 6725
+Wire Wire Line
+	8850 6725 8850 6475
+Connection ~ 8850 6725
+$Comp
+L Connector:TestPoint STOP1
+U 1 1 6219D120
+P 19675 7800
+F 0 "STOP1" H 19733 7918 50  0000 L CNN
+F 1 "TestPoint" H 19733 7827 50  0000 L CNN
+F 2 "TestPoint:TestPoint_THTPad_2.5x2.5mm_Drill1.2mm" H 19875 7800 50  0001 C CNN
+F 3 "~" H 19875 7800 50  0001 C CNN
+	1    19675 7800
+	1    0    0    -1
+$EndComp
+Wire Wire Line
+	1675 8600 5300 8600
+Wire Wire Line
+	5525 5925 5525 6675
+Wire Wire Line
+	5300 5925 5525 5925
+$Comp
+L power:GND #PWR0102
+U 1 1 62BF8DD0
+P 5525 6675
+F 0 "#PWR0102" H 5525 6425 50  0001 C CNN
+F 1 "GND" H 5530 6502 50  0000 C CNN
+F 2 "" H 5525 6675 50  0001 C CNN
+F 3 "" H 5525 6675 50  0001 C CNN
+	1    5525 6675
+	1    0    0    -1
+$EndComp
+$Comp
+L Connector_Generic:Conn_01x02 J12
+U 1 1 62C86F46
+P 5500 8500
+F 0 "J12" H 5580 8492 50  0000 L CNN
+F 1 "Conn_01x02" H 5580 8401 50  0000 L CNN
+F 2 "Connector_PinSocket_2.54mm:PinSocket_1x02_P2.54mm_Vertical" H 5500 8500 50  0001 C CNN
+F 3 "~" H 5500 8500 50  0001 C CNN
+	1    5500 8500
+	1    0    0    -1
+$EndComp
+Connection ~ 5300 8500
+Connection ~ 5300 8600
+Wire Wire Line
+	5300 5125 5525 5125
+Connection ~ 5525 5125
+Wire Wire Line
+	5525 5125 5525 5350
+Wire Wire Line
+	5300 5025 5525 5025
+Wire Wire Line
+	5525 5025 5525 5125
+Wire Wire Line
+	1675 4825 2350 4825
+Wire Wire Line
+	1900 5350 1900 5125
+Wire Wire Line
+	1900 5025 1675 5025
+Wire Wire Line
+	1675 5125 1900 5125
+Connection ~ 1900 5125
+Wire Wire Line
+	1900 5125 1900 5025
+$Comp
+L Connector:TestPoint PB0
+U 1 1 62E7B978
+P 6425 5625
+F 0 "PB0" H 6483 5743 50  0000 L CNN
+F 1 "TestPoint" H 6483 5652 50  0000 L CNN
+F 2 "TestPoint:TestPoint_THTPad_2.5x2.5mm_Drill1.2mm" H 6625 5625 50  0001 C CNN
+F 3 "~" H 6625 5625 50  0001 C CNN
+	1    6425 5625
+	1    0    0    -1
+$EndComp
+$Comp
+L Connector:TestPoint PC4
+U 1 1 62E7CF6C
+P 6950 5625
+F 0 "PC4" H 7008 5743 50  0000 L CNN
+F 1 "TestPoint" H 7008 5652 50  0000 L CNN
+F 2 "TestPoint:TestPoint_THTPad_2.5x2.5mm_Drill1.2mm" H 7150 5625 50  0001 C CNN
+F 3 "~" H 7150 5625 50  0001 C CNN
+	1    6950 5625
+	1    0    0    -1
+$EndComp
+$Comp
+L Connector:TestPoint PC5
+U 1 1 62E7D3A8
+P 7475 5625
+F 0 "PC5" H 7533 5743 50  0000 L CNN
+F 1 "TestPoint" H 7533 5652 50  0000 L CNN
+F 2 "TestPoint:TestPoint_THTPad_2.5x2.5mm_Drill1.2mm" H 7675 5625 50  0001 C CNN
+F 3 "~" H 7675 5625 50  0001 C CNN
+	1    7475 5625
+	1    0    0    -1
+$EndComp
+Wire Wire Line
+	6425 6525 6425 5625
+Wire Wire Line
+	5300 7125 6950 7125
+Wire Wire Line
+	6950 7125 6950 5625
+Connection ~ 5300 7125
+Wire Wire Line
+	5300 7025 7475 7025
+Wire Wire Line
+	7475 7025 7475 5625
+Connection ~ 5300 7025
+Wire Wire Line
+	1675 6525 5300 6525
+Wire Wire Line
+	5300 6525 6425 6525
+Connection ~ 5300 6525
 $EndSCHEMATC

Commit message: New OSHPark manuf candidate.
Parts:
- Q1: footprint Package_TO_SOT_THT:TO-92_HandSolder -> Package_TO_SOT_THT:TO-92_Inline_Wide
Changed lines of the file:
@@
 F 0 "Q1" H 15940 10946 50  0000 L CNN
 F 1 "2N3904" H 15940 10855 50  0000 L CNN
-F 2 "Package_TO_SOT_THT:TO-92_HandSolder" H 15950 10825 50  0001 L CIN
+F 2 "Package_TO_SOT_THT:TO-92_Inline_Wide" H 15950 10825 50  0001 L CIN
 F 3 "https://www.onsemi.com/pub/Collateral/2N3903-D.PDF" H 15750 10900 50  0001 L CNN
 	1    15750 10900

Commit message: New OSHPark manuf candidate.
Parts:
- C6, C8: footprint Capacitor_THT:C_Radial_D6.3mm_H7.0mm_P2.50mm -> Capacitor_THT:CP_Radial_D6.3mm_P2.50mm
Changed lines of the file:
@@
 F 0 "C6" V 4845 3450 50  0000 C CNN
 F 1 "100u" V 4936 3450 50  0000 C CNN
-F 2 "Capacitor_THT:C_Radial_D6.3mm_H7.0mm_P2.50mm" H 5138 3300 50  0001 C CNN
+F 2 "Capacitor_THT:CP_Radial_D6.3mm_P2.50mm" H 5138 3300 50  0001 C CNN
 F 3 "~" H 5100 3450 50  0001 C CNN
 	1    5100 3450
@@
 F 0 "C8" V 4845 4050 50  0000 C CNN
 F 1 "100u" V 4936 4050 50  0000 C CNN
-F 2 "Capacitor_THT:C_Radial_D6.3mm_H7.0mm_P2.50mm" H 5138 3900 50  0001 C CNN
+F 2 "Capacitor_THT:CP_Radial_D6.3mm_P2.50mm" H 5138 3900 50  0001 C CNN
 F 3 "~" H 5100 4050 50  0001 C CNN
 	1    5100 4050
